Commit message: investigate why publisher doesn't work. Start porting work

File: rcomv_uav/urdf/firefly.xacro (robot description, xacro)
@@ -38,5 +38,5 @@
   <xacro:property name="rotor_drag_coefficient" value="8.06428e-05" />
   <xacro:property name="rolling_moment_coefficient" value="0.000001" />
-  <xacro:property name="color" value="$(arg color)" /> <!-- base color -->
+  <xacro:property name="color" value="Black"/> <!-- base color -->
   <!-- Property Blocks -->
   <xacro:property name="body_inertia">
